File: kicad/projects/16bcfs/ctrl-rom-ctrl/ctrl-rom-ctrl.kicad_pcb (KiCad board)
At the start: 4 copper layers, 0 parts

Commit message: Create the Control Logic Mid-Plane for the emulator
* Closes #140
Parts:
- added C1: 0u1, Capacitor_SMD:C_1206_3216Metric_Pad1.33x1.80mm_HandSolder, B.Cu at (47.0, 48.1)
- added C11: 0u1, Capacitor_SMD:C_1206_3216Metric_Pad1.33x1.80mm_HandSolder, F.Cu at (73.2, 41.7)
- added C12: 0u1, Capacitor_SMD:C_1206_3216Metric_Pad1.33x1.80mm_HandSolder, B.Cu at (94.0, 41.5)
- added C13: 0u1, Capacitor_SMD:C_1206_3216Metric_Pad1.33x1.80mm_HandSolder, F.Cu at (91.2, 41.6)
- added C14: 0u1, Capacitor_SMD:C_1206_3216Metric_Pad1.33x1.80mm_HandSolder, B.Cu at (111.9, 41.6)
- added C15: 0u1, Capacitor_SMD:C_1206_3216Metric_Pad1.33x1.80mm_HandSolder, F.Cu at (73.2, 32.8)
- added C16: 0u1, Capacitor_SMD:C_1206_3216Metric_Pad1.33x1.80mm_HandSolder, B.Cu at (94.0, 32.8)
- added C17: 0u1, Capacitor_SMD:C_1206_3216Metric_Pad1.33x1.80mm_HandSolder, F.Cu at (91.2, 32.8)
- added C18: 0u1, Capacitor_SMD:C_1206_3216Metric_Pad1.33x1.80mm_HandSolder, B.Cu at (111.9, 32.8)
- added C19: 0u1, Capacitor_SMD:C_1206_3216Metric_Pad1.33x1.80mm_HandSolder, B.Cu at (56.4, 48.1)
- added C2: 0u1, Capacitor_SMD:C_1206_3216Metric_Pad1.33x1.80mm_HandSolder, F.Cu at (55.7, 33.3)
- added C20: 0u1, Capacitor_SMD:C_1206_3216Metric_Pad1.33x1.80mm_HandSolder, B.Cu at (34.3, 35.9)
- added C21: 0u1, Capacitor_SMD:C_1206_3216Metric_Pad1.33x1.80mm_HandSolder, F.Cu at (32.1, 62.6)
- added C22: 0u1, Capacitor_SMD:C_1206_3216Metric_Pad1.33x1.80mm_HandSolder, F.Cu at (46.1, 62.6)
- added C23: 0u1, Capacitor_SMD:C_1206_3216Metric_Pad1.33x1.80mm_HandSolder, F.Cu at (43.5, 48.5)
- added C24: 47u, Capacitor_SMD:C_1206_3216Metric_Pad1.33x1.80mm_HandSolder, F.Cu at (108.6, 58.4)
- added C25: 47u, Capacitor_SMD:C_1206_3216Metric_Pad1.33x1.80mm_HandSolder, B.Cu at (31.1, 58.4)
- added C3: 0u1, Capacitor_SMD:C_1206_3216Metric_Pad1.33x1.80mm_HandSolder, B.Cu at (37.4, 48.0)
- added C4: 0u1, Capacitor_SMD:C_1206_3216Metric_Pad1.33x1.80mm_HandSolder, F.Cu at (28.9, 48.6)
- added C5: 0u1, Capacitor_SMD:C_1206_3216Metric_Pad1.33x1.80mm_HandSolder, B.Cu at (74.4, 59.5)
- added C6: 0u1, Capacitor_SMD:C_1206_3216Metric_Pad1.33x1.80mm_HandSolder, F.Cu at (56.2, 48.9)
- added C7: 0u1, Capacitor_SMD:C_1206_3216Metric_Pad1.33x1.80mm_HandSolder, F.Cu at (64.3, 33.4)
- added C8: 0u1, Capacitor_SMD:C_1206_3216Metric_Pad1.33x1.80mm_HandSolder, B.Cu at (93.5, 59.6)
- added C9: 0u1, Capacitor_SMD:C_1206_3216Metric_Pad1.33x1.80mm_HandSolder, B.Cu at (58.4, 32.1)
- added D1: Red, LED_SMD:LED_1206_3216Metric_Pad1.42x1.75mm_HandSolder, F.Cu at (73.0, 65.7)
- added D10: Red, LED_SMD:LED_1206_3216Metric_Pad1.42x1.75mm_HandSolder, F.Cu at (95.9, 65.7)
- added D11: Red, LED_SMD:LED_1206_3216Metric_Pad1.42x1.75mm_HandSolder, F.Cu at (98.4, 65.7)
- added D12: Red, LED_SMD:LED_1206_3216Metric_Pad1.42x1.75mm_HandSolder, F.Cu at (101.0, 65.7)
- added D13: Red, LED_SMD:LED_1206_3216Metric_Pad1.42x1.75mm_HandSolder, F.Cu at (103.5, 65.7)
- added D14: Red, LED_SMD:LED_1206_3216Metric_Pad1.42x1.75mm_HandSolder, F.Cu at (106.0, 65.7)
- added D15: Red, LED_SMD:LED_1206_3216Metric_Pad1.42x1.75mm_HandSolder, F.Cu at (108.6, 65.7)
- added D2: Red, LED_SMD:LED_1206_3216Metric_Pad1.42x1.75mm_HandSolder, F.Cu at (75.6, 65.7)
- added D24: Red, LED_SMD:LED_1206_3216Metric_Pad1.42x1.75mm_HandSolder, F.Cu at (111.1, 65.7)
- added D3: Red, LED_SMD:LED_1206_3216Metric_Pad1.42x1.75mm_HandSolder, F.Cu at (78.1, 65.7)
- added D4: Red, LED_SMD:LED_1206_3216Metric_Pad1.42x1.75mm_HandSolder, F.Cu at (80.6, 65.7)
- added D5: Red, LED_SMD:LED_1206_3216Metric_Pad1.42x1.75mm_HandSolder, F.Cu at (83.2, 65.7)
- added D6: Red, LED_SMD:LED_1206_3216Metric_Pad1.42x1.75mm_HandSolder, F.Cu at (85.7, 65.7)
- added D7: Red, LED_SMD:LED_1206_3216Metric_Pad1.42x1.75mm_HandSolder, F.Cu at (88.3, 65.7)
- added D8: Red, LED_SMD:LED_1206_3216Metric_Pad1.42x1.75mm_HandSolder, F.Cu at (90.8, 65.7)
- added D9: Red, LED_SMD:LED_1206_3216Metric_Pad1.42x1.75mm_HandSolder, F.Cu at (93.3, 65.7)
- added J1: Instruction, Connector_PinHeader_2.54mm:PinHeader_1x16_P2.54mm_Vertical, B.Cu at (69.8, 27.9)
- added J2: Control ROM Address, Connector_PinHeader_2.54mm:PinHeader_1x16_P2.54mm_Vertical, B.Cu at (73.7, 48.3)
- added J3: Raw Address for Pgm ROM, Connector_PinHeader_2.54mm:PinHeader_1x16_P2.54mm_Vertical, B.Cu at (73.7, 27.9)
- added J4: Signal Header, Connector_PinHeader_2.54mm:PinHeader_1x16_P2.54mm_Vertical, B.Cu at (27.9, 27.9)
- added J5: Power, Connector_PinHeader_2.54mm:PinHeader_1x02_P2.54mm_Vertical, B.Cu at (27.9, 57.1)
- added J6: Power, Connector_PinHeader_2.54mm:PinHeader_1x02_P2.54mm_Vertical, B.Cu at (111.8, 57.1)
- added R1: 1K, Resistor_SMD:R_1206_3216Metric_Pad1.30x1.75mm_HandSolder, B.Cu at (73.0, 65.8)
- added R10: 1K, Resistor_SMD:R_1206_3216Metric_Pad1.30x1.75mm_HandSolder, B.Cu at (95.9, 65.8)
- added R11: 1K, Resistor_SMD:R_1206_3216Metric_Pad1.30x1.75mm_HandSolder, B.Cu at (98.4, 65.8)
- added R12: 1K, Resistor_SMD:R_1206_3216Metric_Pad1.30x1.75mm_HandSolder, B.Cu at (101.0, 65.8)
- added R13: 1K, Resistor_SMD:R_1206_3216Metric_Pad1.30x1.75mm_HandSolder, B.Cu at (103.5, 65.8)
- added R14: 1K, Resistor_SMD:R_1206_3216Metric_Pad1.30x1.75mm_HandSolder, B.Cu at (106.0, 65.8)
- added R15: 1K, Resistor_SMD:R_1206_3216Metric_Pad1.30x1.75mm_HandSolder, B.Cu at (108.6, 65.8)
- added R16: 0R, Resistor_SMD:R_1206_3216Metric_Pad1.30x1.75mm_HandSolder, F.Cu at (42.6, 56.9)
- added R17: 0R, Resistor_SMD:R_1206_3216Metric_Pad1.30x1.75mm_HandSolder, F.Cu at (45.1, 56.9)
- added R18: 0R, Resistor_SMD:R_1206_3216Metric_Pad1.30x1.75mm_HandSolder, B.Cu at (64.7, 48.6)
- added R19: 0R, Resistor_SMD:R_1206_3216Metric_Pad1.30x1.75mm_HandSolder, B.Cu at (64.7, 45.9)
- added R2: 1K, Resistor_SMD:R_1206_3216Metric_Pad1.30x1.75mm_HandSolder, B.Cu at (75.6, 65.8)
- added R20: 0R, Resistor_SMD:R_1206_3216Metric_Pad1.30x1.75mm_HandSolder, F.Cu at (47.6, 56.9)
- added R21: 0R, Resistor_SMD:R_1206_3216Metric_Pad1.30x1.75mm_HandSolder, B.Cu at (64.7, 51.3)
- added R22: 0R, Resistor_SMD:R_1206_3216Metric_Pad1.30x1.75mm_HandSolder, F.Cu at (65.2, 63.9)
- added R23: 0R, Resistor_SMD:R_1206_3216Metric_Pad1.30x1.75mm_HandSolder, F.Cu at (65.2, 61.4)
- added R24: 1K, Resistor_SMD:R_1206_3216Metric_Pad1.30x1.75mm_HandSolder, B.Cu at (111.1, 65.8)
- added R25: 0R, Resistor_SMD:R_1206_3216Metric_Pad1.30x1.75mm_HandSolder, B.Cu at (48.5, 38.1)
- added R26: 0R, Resistor_SMD:R_1206_3216Metric_Pad1.30x1.75mm_HandSolder, B.Cu at (43.2, 33.3)
- added R27: 0R, Resistor_SMD:R_1206_3216Metric_Pad1.30x1.75mm_HandSolder, F.Cu at (65.2, 66.4)
- added R28: 0R, Resistor_SMD:R_1206_3216Metric_Pad1.30x1.75mm_HandSolder, F.Cu at (59.9, 63.9)
- added R29: 0R, Resistor_SMD:R_1206_3216Metric_Pad1.30x1.75mm_HandSolder, F.Cu at (59.9, 61.4)
- added R3: 1K, Resistor_SMD:R_1206_3216Metric_Pad1.30x1.75mm_HandSolder, B.Cu at (78.1, 65.8)
- added R30: 0R, Resistor_SMD:R_1206_3216Metric_Pad1.30x1.75mm_HandSolder, F.Cu at (59.9, 66.4)
- added R31: 0R, Resistor_SMD:R_1206_3216Metric_Pad1.30x1.75mm_HandSolder, F.Cu at (33.7, 56.9)
- added R32: 0R, Resistor_SMD:R_1206_3216Metric_Pad1.30x1.75mm_HandSolder, F.Cu at (39.1, 56.9)
- added R33: 0R, Resistor_SMD:R_1206_3216Metric_Pad1.30x1.75mm_HandSolder, F.Cu at (36.4, 56.9)
- added R34: 0R, Resistor_SMD:R_1206_3216Metric_Pad1.30x1.75mm_HandSolder, B.Cu at (38.4, 63.5)
- added R35: 0R, Resistor_SMD:R_1206_3216Metric_Pad1.30x1.75mm_HandSolder, B.Cu at (41.1, 63.5)
- added R36: 0R, Resistor_SMD:R_1206_3216Metric_Pad1.30x1.75mm_HandSolder, B.Cu at (35.7, 63.5)
- added R4: 1K, Resistor_SMD:R_1206_3216Metric_Pad1.30x1.75mm_HandSolder, B.Cu at (80.6, 65.8)
- added R5: 1K, Resistor_SMD:R_1206_3216Metric_Pad1.30x1.75mm_HandSolder, B.Cu at (83.2, 65.8)
- added R6: 1K, Resistor_SMD:R_1206_3216Metric_Pad1.30x1.75mm_HandSolder, B.Cu at (85.7, 65.8)
- added R7: 1K, Resistor_SMD:R_1206_3216Metric_Pad1.30x1.75mm_HandSolder, B.Cu at (88.3, 65.8)
- added R8: 1K, Resistor_SMD:R_1206_3216Metric_Pad1.30x1.75mm_HandSolder, B.Cu at (90.8, 65.8)
- added R9: 1K, Resistor_SMD:R_1206_3216Metric_Pad1.30x1.75mm_HandSolder, B.Cu at (93.3, 65.8)
- added U1: 74HC08, Package_SO:SOIC-14_3.9x8.7mm_P1.27mm, B.Cu at (47.8, 54.4)
- added U11: 74HC157, Package_SO:SOIC-16_3.9x9.9mm_P1.27mm, F.Cu at (79.8, 42.5)
- added U12: 74HC157, Package_SO:SOIC-16_3.9x9.9mm_P1.27mm, B.Cu at (87.4, 42.5)
- added U13: 74HC157, Package_SO:SOIC-16_3.9x9.9mm_P1.27mm, F.Cu at (97.8, 42.5)
- added U14: 74HC157, Package_SO:SOIC-16_3.9x9.9mm_P1.27mm, B.Cu at (105.4, 42.5)
- added U15: 74HC193, Package_SO:SOIC-16_3.9x9.9mm_P1.27mm, F.Cu at (79.8, 33.7)
- added U16: 74HC193, Package_SO:SOIC-16_3.9x9.9mm_P1.27mm, B.Cu at (87.4, 33.7)
- added U17: 74HC193, Package_SO:SOIC-16_3.9x9.9mm_P1.27mm, F.Cu at (97.8, 33.7)
- added U18: 74HC193, Package_SO:SOIC-16_3.9x9.9mm_P1.27mm, B.Cu at (105.4, 33.7)
- added U19: 74HC04, Package_SO:SOIC-14_3.9x8.7mm_P1.27mm, B.Cu at (57.2, 54.4)
- added U2: 74HC74, Package_SO:SOIC-14_3.9x8.7mm_P1.27mm, F.Cu at (54.9, 39.3)
- added U21: 74HC08, Package_SO:SOIC-14_3.9x8.7mm_P1.27mm, F.Cu at (38.1, 63.5)
- added U22: 74HC08, Package_SO:SOIC-14_3.9x8.7mm_P1.27mm, F.Cu at (52.1, 63.5)
- added U23: 74HC32, Package_SO:SOIC-14_3.9x8.7mm_P1.27mm, F.Cu at (49.5, 49.5)
- added U3: 74HC03, Package_SO:SOIC-14_3.9x8.7mm_P1.27mm, B.Cu at (38.3, 54.4)
- added U4: 74HC193, Package_SO:SOIC-16_3.9x9.9mm_P1.27mm, F.Cu at (35.6, 49.5)
- added U5: 74HC541, Package_SO:SOIC-20W_7.5x12.8mm_P1.27mm, B.Cu at (82.5, 56.5)
- added U6: 74HC00, Package_SO:SOIC-14_3.9x8.7mm_P1.27mm, F.Cu at (62.2, 49.7)
- added U7: 74HC00, Package_SO:SOIC-14_3.9x8.7mm_P1.27mm, F.Cu at (63.4, 39.4)
- added U8: 74HC541, Package_SO:SOIC-20W_7.5x12.8mm_P1.27mm, B.Cu at (101.6, 56.5)
- added U9: 74HC165, Package_SO:SOIC-16_3.9x9.9mm_P1.27mm, B.Cu at (59.3, 38.7)
- added X1: XO32, eryjus:Oscillator_DIP-8-14, F.Cu at (31.8, 41.9)
Routing:
- net GNDREF: track 0.00 -> 612.9 mm, vias 0 -> 105
- net VCC: track 0.00 -> 303.4 mm, vias 0 -> 39
- net ~{QR}: track 0.00 -> 184.6 mm, vias 0 -> 2
- net ~{DONE}: track 0.00 -> 123.5 mm, vias 0 -> 8
- net CPY_CLK: track 0.00 -> 110.1 mm, vias 0 -> 1
- net SRAM ~{CE}: track 0.00 -> 100.7 mm, vias 0 -> 2
- net ~{Raw_Cpy_Clk}: track 0.00 -> 89.5 mm, vias 0 -> 4
- net ~{RESET}: track 0.00 -> 72.2 mm, vias 0 -> 2
- net QS: track 0.00 -> 71.9 mm, vias 0 -> 4
- net Addr Counter ~{CO}: track 0.00 -> 71.4 mm, vias 0 -> 3
- net QC: track 0.00 -> 64.5 mm, vias 0 -> 8
- net RAW_CPY_CLK: track 0.00 -> 61.7 mm, vias 0 -> 2
- net Net-(U19-Pad13): track 0.00 -> 60.3 mm, vias 0 -> 3
- net INSTR_AC: track 0.00 -> 56.1 mm, vias 0 -> 3
- net INSTR_AE: track 0.00 -> 54.2 mm, vias 0 -> 1
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- added copper zone on B.Cu, net GNDREF
- added copper zone on F.Cu, net GNDREF
- added copper zone on In1.Cu, net GNDREF
- added copper zone on In2.Cu, net VCC
Other:
- board outline added: 88.9 x 43.2 mm
- board text added: "0R"
- board text added: "0u1"
- board text added: "16-Bit Computer From Scratch"
- board text added: "47u"
- board text added: "74HC00"
- board text added: "74HC03"
- board text added: "74HC04"
- board text added: "74HC08"
- board text added: "74HC157"
- board text added: "74HC165"
- board text added: "74HC193"
- board text added: "74HC32"
- board text added: "74HC541"
- board text added: "74HC74"
- board text added: "A"
- board text added: "AND3C"
- board text added: "AND3D"
- board text added: "B"
- board text added: "Control ROM Control Module"
- board text added: "Ctrl ROM Address"
- board text added: "ERYJUS"
- board text added: "GND"
- board text added: "Instruction"
- board text added: "Local Xtal"
- board text added: "NAND2C"
- board text added: "Raw Addr for Pgm ROM"
- board text added: "Raw Sys Clk"
- board text added: "Signals"
- board text added: "VCC"
- board text added: "VCC GND"
- board text added: "Y"
- board text added: "oNANDB"
- board text added: "oNANDC"
- board text added: "oNANDD"
- board text added: "v1.0"
