File: kicad/projects/16bcfs/reset/state.kicad_sch (KiCad schematic)
At the start: 9 parts, among them U4 74HC00, U6 74HC00, U7 74HC02, U8 74HC123, U9 74HC03

Commit message: Address some issues with the Reset Logic
There were a couple of fixes.  One in relation to how the 74xx123 IC was
emulated and others to the schematic to address issues in real life in
the breadboard prototype.
Parts:
- R10, R8: value 100R -> 10k
Connections:
- net GNDREF: no longer U8.11 (Clr), U8.3 (Clr)
- net VCC: now also U8.11 (Clr), U8.3 (Clr)
Changed lines of the file:
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@@
   (junction (at 33.02 62.23) (diameter 0) (color 0 0 0 0)
   )
-  (junction (at 31.75 146.05) (diameter 0) (color 0 0 0 0)
-  )
   (junction (at 109.22 110.49) (diameter 0) (color 0 0 0 0)
   )
@@
   (junction (at 111.76 106.68) (diameter 0) (color 0 0 0 0)
   )
+  (junction (at 16.51 54.61) (diameter 0) (color 0 0 0 0)
+  )
   (junction (at 106.68 101.6) (diameter 0) (color 0 0 0 0)
   )
-  (junction (at 33.02 90.17) (diameter 0) (color 0 0 0 0)
+  (junction (at 16.51 109.22) (diameter 0) (color 0 0 0 0)
   )
   (no_connect (at 60.96 128.27))
@@
     (stroke (width 0) (type default))
   )
-  (wire (pts (xy 31.75 146.05) (xy 31.75 148.59))
+  (wire (pts (xy 31.75 125.73) (xy 31.75 148.59))
     (stroke (width 0) (type default))
   )
@@
     (stroke (width 0) (type default))
   )
+  (wire (pts (xy 16.51 109.22) (xy 31.75 109.22))
+    (stroke (width 0) (type default))
+  )
   (wire (pts (xy 35.56 116.84) (xy 31.75 116.84))
     (stroke (width 0) (type default))
@@
     (stroke (width 0) (type default))
   )
-  (wire (pts (xy 48.26 135.89) (xy 48.26 146.05))
+  (wire (pts (xy 48.26 135.89) (xy 48.26 137.16))
     (stroke (width 0) (type default))
   )
@@
     (stroke (width 0) (type default))
   )
+  (wire (pts (xy 16.51 137.16) (xy 48.26 137.16))
+    (stroke (width 0) (type default))
+  )
   (wire (pts (xy 168.91 142.24) (xy 217.17 142.24))
     (stroke (width 0) (type default))
@@
     (stroke (width 0) (type default))
   )
-  (wire (pts (xy 33.02 71.12) (xy 33.02 90.17))
+  (wire (pts (xy 33.02 71.12) (xy 33.02 92.71))
     (stroke (width 0) (type default))
   )
@@
     (stroke (width 0) (type default))
   )
-  (wire (pts (xy 33.02 90.17) (xy 33.02 92.71))
-    (stroke (width 0) (type default))
-  )
   (wire (pts (xy 93.98 80.01) (xy 147.32 80.01))
     (stroke (width 0) (type default))
@@
     (stroke (width 0) (type default))
   )
+  (wire (pts (xy 16.51 54.61) (xy 33.02 54.61))
+    (stroke (width 0) (type default))
+  )
   (wire (pts (xy 172.72 38.1) (xy 176.53 38.1))
     (stroke (width 0) (type default))
@@
     (stroke (width 0) (type default))
   )
-  (wire (pts (xy 33.02 53.34) (xy 33.02 54.61))
+  (wire (pts (xy 16.51 53.34) (xy 16.51 54.61))
     (stroke (width 0) (type default))
   )
@@
     (stroke (width 0) (type default))
   )
-  (wire (pts (xy 48.26 146.05) (xy 31.75 146.05))
-    (stroke (width 0) (type default))
-  )
   (wire (pts (xy 167.64 88.9) (xy 167.64 101.6))
     (stroke (width 0) (type default))
@@
     (stroke (width 0) (type default))
   )
-  (wire (pts (xy 31.75 125.73) (xy 31.75 146.05))
+  (wire (pts (xy 16.51 109.22) (xy 16.51 137.16))
     (stroke (width 0) (type default))
   )
@@
     (stroke (width 0) (type default))
   )
+  (wire (pts (xy 16.51 54.61) (xy 16.51 82.55))
+    (stroke (width 0) (type default))
+  )
   (wire (pts (xy 93.98 115.57) (xy 93.98 120.65))
     (stroke (width 0) (type default))
@@
     (stroke (width 0) (type default))
   )
-  (wire (pts (xy 49.53 81.28) (xy 49.53 90.17))
-    (stroke (width 0) (type default))
-  )
-  (wire (pts (xy 31.75 107.95) (xy 31.75 109.22))
+  (wire (pts (xy 49.53 81.28) (xy 49.53 82.55))
+    (stroke (width 0) (type default))
+  )
+  (wire (pts (xy 16.51 107.95) (xy 16.51 109.22))
     (stroke (width 0) (type default))
   )
@@
     (stroke (width 0) (type default))
   )
+  (wire (pts (xy 16.51 82.55) (xy 49.53 82.55))
+    (stroke (width 0) (type default))
+  )
   (wire (pts (xy 82.55 115.57) (xy 93.98 115.57))
     (stroke (width 0) (type default))
@@
   )
   (wire (pts (xy 144.78 54.61) (xy 147.32 54.61))
-    (stroke (width 0) (type default))
-  )
-  (wire (pts (xy 49.53 90.17) (xy 33.02 90.17))
     (stroke (width 0) (type default))
   )
@@
     )
   )
-  (symbol (lib_id "power:VCC") (at 33.02 53.34 0) (unit 1)
+  (symbol (lib_id "power:VCC") (at 16.51 53.34 0) (unit 1)
     (in_bom yes) (on_board yes) (dnp no) (fields_autoplaced)
-    (property "Reference" "#PWR019" (at 33.02 57.15 0)
-      (effects (font (size 1.27 1.27)) hide)
-    )
-    (property "Value" "VCC" (at 33.02 48.26 0)
+    (property "Reference" "#PWR019" (at 16.51 57.15 0)
+      (effects (font (size 1.27 1.27)) hide)
+    )
+    (property "Value" "VCC" (at 16.51 48.26 0)
       (effects (font (size 1.27 1.27)))
     )
-    (property "Footprint" "" (at 33.02 53.34 0)
-      (effects (font (size 1.27 1.27)) hide)
-    )
-    (property "Datasheet" "" (at 33.02 53.34 0)
+    (property "Footprint" "" (at 16.51 53.34 0)
+      (effects (font (size 1.27 1.27)) hide)
+    )
+    (property "Datasheet" "" (at 16.51 53.34 0)
       (effects (font (size 1.27 1.27)) hide)
     )
@@
     )
   )
-  (symbol (lib_id "power:VCC") (at 31.75 107.95 0) (unit 1)
+  (symbol (lib_id "power:VCC") (at 16.51 107.95 0) (unit 1)
     (in_bom yes) (on_board yes) (dnp no) (fields_autoplaced)
-    (property "Reference" "#PWR022" (at 31.75 111.76 0)
-      (effects (font (size 1.27 1.27)) hide)
-    )
-    (property "Value" "VCC" (at 31.75 102.87 0)
+    (property "Reference" "#PWR022" (at 16.51 111.76 0)
+      (effects (font (size 1.27 1.27)) hide)
+    )
+    (property "Value" "VCC" (at 16.51 102.87 0)
       (effects (font (size 1.27 1.27)))
     )
-    (property "Footprint" "" (at 31.75 107.95 0)
-      (effects (font (size 1.27 1.27)) hide)
-    )
-    (property "Datasheet" "" (at 31.75 107.95 0)
+    (property "Footprint" "" (at 16.51 107.95 0)
+      (effects (font (size 1.27 1.27)) hide)
+    )
+    (property "Datasheet" "" (at 16.51 107.95 0)
       (effects (font (size 1.27 1.27)) hide)
     )
@@
       (effects (font (size 1.27 1.27)) (justify left))
     )
-    (property "Value" "100R" (at 25.4 113.665 0)
+    (property "Value" "10k" (at 25.4 113.665 0)
       (effects (font (size 1.27 1.27)) (justify left))
     )
@@
       (effects (font (size 1.27 1.27)) (justify left))
     )
-    (property "Value" "100R" (at 26.67 59.055 0)
-      (effects (font (size 1.27 1.27)) (justify left))
-    )
+    (property "Value" "10k" (at 26.67 59.055 0)
+      (effects (font (size 1.27 1.27)) (justify left))
+    )

Commit message: Update the Reset Module
This commit updates the reset module to reflect the changes made on the
breadboard which stabilized the build.
Connections:
- net VCC: now also U8.2 (B); no longer U8.3 (Clr)
- net ~{CPYHLD}: now also U8.3 (Clr); no longer U8.2 (B)
Changed lines of the file:
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@@
     (stroke (width 0) (type default))
   )
-  (wire (pts (xy 16.51 54.61) (xy 16.51 82.55))
+  (wire (pts (xy 16.51 54.61) (xy 16.51 73.66))
     (stroke (width 0) (type default))
   )
@@
   )
   (wire (pts (xy 144.78 40.64) (xy 144.78 44.45))
+    (stroke (width 0) (type default))
+  )
+  (wire (pts (xy 24.13 83.82) (xy 49.53 83.82))
     (stroke (width 0) (type default))
   )
@@
     (stroke (width 0) (type default))
   )
-  (wire (pts (xy 49.53 81.28) (xy 49.53 82.55))
+  (wire (pts (xy 49.53 81.28) (xy 49.53 83.82))
     (stroke (width 0) (type default))
   )
@@
     (stroke (width 0) (type default))
   )
-  (wire (pts (xy 16.51 82.55) (xy 49.53 82.55))
-    (stroke (width 0) (type default))
-  )
   (wire (pts (xy 82.55 115.57) (xy 93.98 115.57))
     (stroke (width 0) (type default))
@@
     (stroke (width 0) (type default))
   )
-  (wire (pts (xy 27.94 73.66) (xy 36.83 73.66))
+  (wire (pts (xy 16.51 73.66) (xy 36.83 73.66))
     (stroke (width 0) (type default))
   )
@@
     (effects (font (size 1.27 1.27)) (justify right))
   )
-  (hierarchical_label "~{CPYHLD}" (shape input) (at 27.94 73.66 180) (fields_autoplaced)
+  (hierarchical_label "~{CPYHLD}" (shape input) (at 24.13 83.82 180) (fields_autoplaced)
     (effects (font (size 1.27 1.27)) (justify right))
   )
