File: kicad/projects/16bcfs/clock-module/state.kicad_sch (KiCad schematic)
At the start: 10 parts, among them SW6 Oscillator, SW7 Adjustable Clock, SW8 Single Step, U1 74HC00, U2 74HC00, U5 74HC02, U6 74HC08

Commit message: Clean up the Reset and Clock Modules
Connections:
- net Step_Sel: now also U2.11, U2.9; no longer U2.12, U2.8
- net at U5.13: now also U2.12; no longer U2.9
- net at U5.10: now also U2.10; no longer U2.13
- new net ~{StepSel}: U2.13, U2.8
Other:
- moved on the sheet: U2C, U2D
Changed lines of the file:
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@@
   (junction (at 175.26 46.99) (diameter 0) (color 0 0 0 0)
   )
+  (junction (at 180.34 151.13) (diameter 0) (color 0 0 0 0)
+  )
   (junction (at 123.19 115.57) (diameter 0) (color 0 0 0 0)
   )
@@
     (stroke (width 0) (type default))
   )
+  (wire (pts (xy 180.34 151.13) (xy 187.96 151.13))
+    (stroke (width 0) (type default))
+  )
   (wire (pts (xy 130.81 134.62) (xy 57.15 134.62))
     (stroke (width 0) (type default))
@@
   (wire (pts (xy 149.86 132.08) (xy 146.05 132.08))
     (stroke (width 0) (type default))
+  )
+  (hierarchical_label "~{StepSel}" (shape output) (at 187.96 151.13 0) (fields_autoplaced)
+    (effects (font (size 1.27 1.27)) (justify left))
   )
   (hierarchical_label "Adj_Sel" (shape output) (at 187.96 91.44 0) (fields_autoplaced)
@@
     )
   )
-  (symbol (lib_id "74xx:74HC00") (at 166.37 132.08 0) (unit 3)
-    (in_bom yes) (on_board yes) (dnp no)
-    (property "Reference" "U2" (at 162.56 130.175 0)
-      (effects (font (size 1.27 1.27)) (justify left))
-    )
-    (property "Value" "74HC00" (at 162.56 132.08 0)
-      (effects (font (size 1.27 1.27)) (justify left))
-    )
-    (property "Footprint" "" (at 166.37 132.08 0)
-      (effects (font (size 1.27 1.27)) hide)
-    )
-    (property "Datasheet" "http://www.ti.com/lit/gpn/sn74hc00" (at 166.37 132.08 0)
+  (symbol (lib_id "74xx:74HC00") (at 166.37 151.13 0) (unit 3)
+    (in_bom yes) (on_board yes) (dnp no)
+    (property "Reference" "U2" (at 162.56 149.225 0)
+      (effects (font (size 1.27 1.27)) (justify left))
+    )
+    (property "Value" "74HC00" (at 162.56 151.13 0)
+      (effects (font (size 1.27 1.27)) (justify left))
+    )
+    (property "Footprint" "" (at 166.37 151.13 0)
+      (effects (font (size 1.27 1.27)) hide)
+    )
+    (property "Datasheet" "http://www.ti.com/lit/gpn/sn74hc00" (at 166.37 151.13 0)
       (effects (font (size 1.27 1.27)) hide)
     )
@@
     )
   )
-  (symbol (lib_id "74xx:74HC00") (at 166.37 151.13 0) (unit 4)
-    (in_bom yes) (on_board yes) (dnp no)
-    (property "Reference" "U2" (at 162.56 149.225 0)
-      (effects (font (size 1.27 1.27)) (justify left))
-    )
-    (property "Value" "74HC00" (at 162.56 151.13 0)
-      (effects (font (size 1.27 1.27)) (justify left))
-    )
-    (property "Footprint" "" (at 166.37 151.13 0)
-      (effects (font (size 1.27 1.27)) hide)
-    )
-    (property "Datasheet" "http://www.ti.com/lit/gpn/sn74hc00" (at 166.37 151.13 0)
-      (effects (font (size 1.27 1.27)) hide)
-    )
+  (symbol (lib_id "74xx:74HC00") (at 166.37 132.08 0) (unit 4)
+    (in_bom yes) (on_board yes) (dnp no)
+    (property "Reference" "U2" (at 162.56 130.175 0)
+      (effects (font (size 1.27 1.27)) (justify left))
+    )
+    (property "Value" "74HC00" (at 162.56 132.08 0)
+      (effects (font (size 1.27 1.27)) (justify left))
+    )
+    (property "Footprint" "" (at 166.37 132.08 0)
+      (effects (font (size 1.27 1.27)) hide)
+    )
+    (property "Datasheet" "http://www.ti.com/lit/gpn/sn74hc00" (at 166.37 132.08 0)
+      (effects (font (size 1.27 1.27)) hide)
+    )
