File: kicad/projects/16bcfs/control-logic-midplane/control-logic-midplane.kicad_sch (KiCad schematic)
At the start: 215 parts, among them J1 Addr Bus 1 Assert & Control, J10 Control Pins 3, J11 Ctrl4 Address Pins, J12 Control Pins 4, J13 Ctrl5 Address Pins, J14 Control Pins 5, J15 Ctrl6 Address Pins, J16 Control Pins 6, J17 Signal Pins 0, J18 Signal Pins 1, J19 Signal Pins 2, J2 ALU Control (2), J20 Signal Pins 3, J21 Signal Pins 4, J22 Signal Pins 5, J23 Signal Pins 6, J24 Registers (2), J25 ALU Control, J26 Power Socket, J27 R1 Connector, J28 R7 Connector, J29 PgmPC Connector, J3 Ctrl0 Address Pins, J30 Device/Control 01/02, J31 Ctrl9 Address Pins, J32 Control Pins 9, J33 CtrlA Address Pins, J34 Control Pins A, J35 CtrlB Address Pins, J36 Control Pins B, J37 Ctrl7 Address Pins, J38 Control Pins 7, J39 Ctrl8 Address Pins, J4 Control Pins 0, J40 Control Pins 8, J41 R2 Connector, J42 R8 Connector, J43 PgmRA Connector, J44 Instruction Register Input, J45 Device/Control 03/04, J46 Signal Pins 9, J47 Signal Pins A, J48 Signal Pins B, J49 Signal Pins 7, J5 Ctrl1 Address Pins, J50 Signal Pins 8, J51 R3 Connector, J52 R9 Connector, J53 PgmSP Connector, J54 Device/Control 05/06, J55 Pgm ROM Address Copy, J56 R10 Connector, J57 IntPC Connector, J58 R4 Connector, J59 Power, J6 Control Pins 1, J60 CtrlE Address Pins, J61 Control Pins E, J62 CtrlF Address Pins, J63 Control Pins F, J64 CtrlC Address Pins, J65 Control Pins C, J66 CtrlD Address Pins, J67 Control Pins D, J68 Power, J69 Instruction Register Input, J7 Ctrl2 Address Pins, J70 R5 Connector, J71 R11 Connector, J72 IntRA Connector, J73 Device/Control 07/08, J74 Signal Pins E, J75 Signal Pins F, J76 Signal Pins C, J77 Signal Pins D, J78 Raw Address for Pgm ROM, J79 Control ROM Address, J8 Control Pins 2, J80 R6 Connector, J81 R12 Connector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

Commit message: Rename #RHLD to #CPYHLD on the Ctrl Rom Ctrl & Midplane
The logic for the signal does not change, but the purpose does.  The
Reset Circuit will handle the #RHLD now, but it needs to know when the
copy is complete.
Connections:
- net ~{RHLD} renamed ~{CPYHLD}
Changed lines of the file:
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@@
     )
   )
-  (global_label "~{RHLD}" (shape output) (at 537.845 538.48 180) (fields_autoplaced)
-    (effects (font (size 1.27 1.27)) (justify right))
-    (property "Intersheetrefs" "${INTERSHEET_REFS}" (at 529.9612 538.48 0)
+  (global_label "~{CPYHLD}" (shape output) (at 537.845 538.48 180) (fields_autoplaced)
+    (effects (font (size 1.27 1.27)) (justify right))
+    (property "Intersheetrefs" "${INTERSHEET_REFS}" (at 527.6026 538.48 0)
       (effects (font (size 1.27 1.27)) (justify right) hide)
     )
@@
     )
   )
-  (global_label "~{RHLD}" (shape input) (at 848.36 59.055 0) (fields_autoplaced)
-    (effects (font (size 1.27 1.27)) (justify left))
-    (property "Intersheetrefs" "${INTERSHEET_REFS}" (at 856.2438 59.055 0)
-      (effects (font (size 1.27 1.27)) (justify left) hide)
-    )
+  (global_label "~{CPYHLD}" (shape input) (at 848.36 59.055 0) (fields_autoplaced)
+    (effects (font (size 1.27 1.27)) (justify left))
+    (property "Intersheetrefs" "${INTERSHEET_REFS}" (at 858.6024 59.055 0)
+      (effects (font (size 1.27 1.27)) (justify left) hide)
+    )

Commit message: Schematic changes for clock and control ROM
Connections:
- net RAW_SYS_CLK renamed HS_CLK
Changed lines of the file:
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@@
     )
   )
-  (global_label "RAW_SYS_CLK" (shape input) (at 537.845 551.18 180) (fields_autoplaced)
-    (effects (font (size 1.27 1.27)) (justify right))
-    (property "Intersheetrefs" "${INTERSHEET_REFS}" (at 522.0389 551.18 0)
+  (global_label "HS_CLK" (shape input) (at 537.845 551.18 180) (fields_autoplaced)
+    (effects (font (size 1.27 1.27)) (justify right))
+    (property "Intersheetrefs" "${INTERSHEET_REFS}" (at 527.7841 551.18 0)
       (effects (font (size 1.27 1.27)) (justify right) hide)
     )
@@
     )
   )
-  (global_label "RAW_SYS_CLK" (shape output) (at 848.36 64.135 0) (fields_autoplaced)
-    (effects (font (size 1.27 1.27)) (justify left))
-    (property "Intersheetrefs" "${INTERSHEET_REFS}" (at 864.1661 64.135 0)
-      (effects (font (size 1.27 1.27)) (justify left) hide)
-    )
+  (global_label "HS_CLK" (shape output) (at 848.36 64.135 0) (fields_autoplaced)
+    (effects (font (size 1.27 1.27)) (justify left))
+    (property "Intersheetrefs" "${INTERSHEET_REFS}" (at 858.4209 64.135 0)
+      (effects (font (size 1.27 1.27)) (justify left) hide)
+    )
