File: kicad/projects/16bcfs/fetch-register/fetch-register.kicad_sch (KiCad schematic)
At the start: 118 parts, among them J1 InstrRegInput, J2 ALU Bus B, J3 FetchBusInput, J4 Main Bus, J5 Control Signals, J6 Address Bus 2, J7 Power, U1 74HC574, U10 74HC574, U11 74HC574, U12 74HC541, U2 74HC574, U3 74HC574, U4 74HC574, U5 74HC574, U6 74HC574, U7 74HC04, U8 74HC574, U9 74HC574

Commit message: Complete the routing for the Fetch Register PCB
This commit completes the routing for the PCB, unless something needs to
move to make room for silkscreen.
Parts:
- added C14: 0.1uF, Capacitor_SMD:C_1206_3216Metric_Pad1.33x1.80mm_HandSolder, symbol Device:C_Polarized_US
Connections:
- net GNDREF: now also C14.2
- net VCC: now also C14.1
Changed lines of the file:
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@@
   (junction (at 371.475 204.47) (diameter 0) (color 0 0 0 0)
   )
+  (junction (at 390.525 196.85) (diameter 0) (color 0 0 0 0)
+  )
   (junction (at 256.54 28.575) (diameter 0) (color 0 0 0 0)
   )
@@
   (junction (at 276.86 73.025) (diameter 0) (color 0 0 0 0)
   )
+  (junction (at 390.525 204.47) (diameter 0) (color 0 0 0 0)
+  )
   (junction (at 371.475 196.85) (diameter 0) (color 0 0 0 0)
   )
@@
     (stroke (width 0) (type default))
   )
+  (wire (pts (xy 390.525 204.47) (xy 401.32 204.47))
+    (stroke (width 0) (type default))
+  )
   (wire (pts (xy 173.355 118.745) (xy 173.355 153.035))
     (stroke (width 0) (type default))
@@
     (stroke (width 0) (type default))
   )
-  (wire (pts (xy 384.175 196.85) (xy 401.32 196.85))
+  (wire (pts (xy 384.175 196.85) (xy 390.525 196.85))
     (stroke (width 0) (type default))
   )
@@
     (stroke (width 0) (type default))
   )
-  (wire (pts (xy 384.175 204.47) (xy 401.32 204.47))
+  (wire (pts (xy 384.175 204.47) (xy 390.525 204.47))
     (stroke (width 0) (type default))
   )
@@
     (stroke (width 0) (type default))
   )
+  (wire (pts (xy 390.525 196.85) (xy 401.32 196.85))
+    (stroke (width 0) (type default))
+  )
   (wire (pts (xy 102.87 217.805) (xy 102.87 221.615))
     (stroke (width 0) (type default))
@@
         )
       )
+    )
+  )
+  (symbol (lib_id "Device:C_Polarized_US") (at 390.525 200.66 0) (unit 1)
+    (in_bom yes) (on_board yes) (dnp no)
+    (property "Reference" "C14" (at 389.255 207.01 0)
+      (effects (font (size 1.27 1.27)) (justify left))
+    )
+    (property "Value" "0.1uF" (at 389.255 209.55 0)
+      (effects (font (size 1.27 1.27)) (justify left))
+    )
+    (property "Footprint" "Capacitor_SMD:C_1206_3216Metric_Pad1.33x1.80mm_HandSolder" (at 390.525 200.66 0)
+      (effects (font (size 1.27 1.27)) hide)
+    )
+    (property "Datasheet" "~" (at 390.525 200.66 0)
+      (effects (font (size 1.27 1.27)) hide)
+    )
+    (pin "1")
+    (pin "2")
+    (instances
+      (project "fetch-register"
+        (path "/d0ae44e5-d74e-4df6-bf3d-e0535c5a7785"
+          (reference "C14") (unit 1)
+        )
+      )

Commit message: Fix the Fetch Register LEDs signal direction
Also changes the Emulator from the pedantic copy mode.
Connections:
- net GNDREF: now also R17.1, R18.1, R19.1, R20.1
- net VCC: no longer R17.1, R18.1, R19.1, R20.1
Other:
- moved on the sheet: C1, C10, C11, C12, C13, C14, C2, C3, C4, C5, C6, C7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

Commit message: Updte LED polarity on the fetch register
Connections:
- net ALU B LED: now also D18.2 (A); no longer D18.1 (K)
- net AddrBus2 LED: now also D19.2 (A); no longer D19.1 (K)
- net InstrReg LED: now also D20.2 (A); no longer D20.1 (K)
- net Main LED: now also D17.2 (A); no longer D17.1 (K)
- net at R18.2: now also D18.1 (K); no longer D18.2 (A)
- net at R19.2: now also D19.1 (K); no longer D19.2 (A)
- net at R20.2: now also D20.1 (K); no longer D20.2 (A)
- net at R17.2: now also D17.1 (K); no longer D17.2 (A)
Changed lines of the file:
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@@
     (stroke (width 0) (type default))
   )
-  (wire (pts (xy 248.92 157.48) (xy 248.92 173.99))
-    (stroke (width 0) (type default))
-  )
   (wire (pts (xy 45.72 229.87) (xy 45.72 232.41))
     (stroke (width 0) (type default))
@@
     (stroke (width 0) (type default))
   )
+  (wire (pts (xy 248.92 157.48) (xy 248.92 173.99))
+    (stroke (width 0) (type default))
+  )
   (wire (pts (xy 127 186.69) (xy 170.18 186.69))
     (stroke (width 0) (type default))
@@
     (stroke (width 0) (type default))
   )
-  (wire (pts (xy 254 157.48) (xy 254 173.99))
-    (stroke (width 0) (type default))
-  )
   (wire (pts (xy 317.5 106.68) (xy 325.12 106.68))
     (stroke (width 0) (type default))
@@
     (stroke (width 0) (type default))
   )
-  (wire (pts (xy 251.46 157.48) (xy 251.46 173.99))
-    (stroke (width 0) (type default))
-  )
   (wire (pts (xy 261.62 212.09) (xy 261.62 224.79))
     (stroke (width 0) (type default))
@@
     (stroke (width 0) (type default))
   )
-  (wire (pts (xy 256.54 157.48) (xy 256.54 173.99))
-    (stroke (width 0) (type default))
-  )
   (wire (pts (xy 87.63 218.44) (xy 87.63 222.25))
     (stroke (width 0) (type default))
@@
     (stroke (width 0) (type default))
   )
+  (wire (pts (xy 256.54 157.48) (xy 256.54 173.99))
+    (stroke (width 0) (type default))
+  )
   (wire (pts (xy 90.17 165.1) (xy 90.17 168.91))
     (stroke (width 0) (type default))
@@
     (stroke (width 0) (type default))
   )
+  (wire (pts (xy 254 157.48) (xy 254 173.99))
+    (stroke (width 0) (type default))
+  )
   (wire (pts (xy 152.4 232.41) (xy 156.21 232.41))
     (stroke (width 0) (type default))
@@
     (stroke (width 0) (type default))
   )
+  (wire (pts (xy 251.46 157.48) (xy 251.46 173.99))
+    (stroke (width 0) (type default))
+  )
   (wire (pts (xy 354.33 111.76) (xy 359.41 111.76))
     (stroke (width 0) (type default))
@@
     )
   )
-  (symbol (lib_id "Device:LED") (at 251.46 153.67 90) (unit 1)
+  (symbol (lib_id "Device:LED") (at 251.46 153.67 90) (mirror x) (unit 1)
     (in_bom yes) (on_board yes) (dnp no) (fields_autoplaced)
-    (property "Reference" "D18" (at 248.92 156.5276 90)
+    (property "Reference" "D18" (at 248.92 150.8124 90)
       (effects (font (size 1.27 1.27)) (justify left) hide)
     )
-    (property "Value" "Red" (at 248.92 153.9876 90)
+    (property "Value" "Red" (at 248.92 153.3524 90)
       (effects (font (size 1.27 1.27)) (justify left) hide)
     )
@@
     )
   )
-  (symbol (lib_id "Device:LED") (at 256.54 153.67 90) (unit 1)
+  (symbol (lib_id "Device:LED") (at 256.54 153.67 90) (mirror x) (unit 1)
     (in_bom yes) (on_board yes) (dnp no) (fields_autoplaced)
-    (property "Reference" "D20" (at 254 156.5276 90)
+    (property "Reference" "D20" (at 254 150.8124 90)
       (effects (font (size 1.27 1.27)) (justify left) hide)
     )
-    (property "Value" "Red" (at 254 153.9876 90)
+    (property "Value" "Red" (at 254 153.3524 90)
       (effects (font (size 1.27 1.27)) (justify left) hide)
     )
@@
     )
   )
-  (symbol (lib_id "Device:LED") (at 248.92 153.67 90) (unit 1)
+  (symbol (lib_id "Device:LED") (at 248.92 153.67 90) (mirror x) (unit 1)
     (in_bom yes) (on_board yes) (dnp no) (fields_autoplaced)
-    (property "Reference" "D17" (at 246.38 156.5276 90)
+    (property "Reference" "D17" (at 246.38 150.8124 90)
       (effects (font (size 1.27 1.27)) (justify left) hide)
     )
-    (property "Value" "Red" (at 246.38 153.9876 90)
+    (property "Value" "Red" (at 246.38 153.3524 90)
       (effects (font (size 1.27 1.27)) (justify left) hide)
     )
@@
     )
   )
-  (symbol (lib_id "Device:LED") (at 254 153.67 90) (unit 1)
+  (symbol (lib_id "Device:LED") (at 254 153.67 90) (mirror x) (unit 1)
     (in_bom yes) (on_board yes) (dnp no) (fields_autoplaced)
-    (property "Reference" "D19" (at 251.46 156.5276 90)
+    (property "Reference" "D19" (at 251.46 150.8124 90)
       (effects (font (size 1.27 1.27)) (justify left) hide)
     )
-    (property "Value" "Red" (at 251.46 153.9876 90)
+    (property "Value" "Red" (at 251.46 153.3524 90)
       (effects (font (size 1.27 1.27)) (justify left) hide)
     )
